Commit message: update moveit config

File: open_manipulator_with_tb3_description/urdf/open_manipulator_with_tb3_waffle.urdf.xacro (robot description, xacro)
@@ -6,4 +6,17 @@
   <!-- Include OpenManipulator Chain Gazebo Parameter -->
   <xacro:include filename="$(find open_manipulator_with_tb3_description)/urdf/open_manipulator_with_tb3.gazebo.xacro" />
+  <!-- Transmission macro -->
+  <xacro:macro name="SimpleTransmission" params="joint n">
+    <transmission name="tran${n}">
+      <type>transmission_interface/SimpleTransmission</type>
+      <joint name="${joint}">
+	      <hardwareInterface>hardware_interface/PositionJointInterface</hardwareInterface>
+      </joint>
+      <actuator name="motor${n}">
+        <hardwareInterface>hardware_interface/PositionJointInterface</hardwareInterface>
+        <mechanicalReduction>1</mechanicalReduction>
+      </actuator>
+    </transmission>
+  </xacro:macro>
   <!-- Base fixed joint -->
   <joint name="base_fixed" type="fixed">
@@ -27,5 +40,5 @@
       </geometry>
     </collision>
-    <inertial>
+    <inertial>z
       <origin xyz="0 0 0" />
       <mass value="0.082" />
@@ -51,14 +64,5 @@
   </joint>
   <!-- Transmission 1 -->
-  <transmission name="tran1">
-    <type>transmission_interface/SimpleTransmission</type>
-    <joint name="joint1">
-      <hardwareInterface>hardware_interface/EffortJointInterface</hardwareInterface>
-    </joint>
-    <actuator name="motor1">
-      <hardwareInterface>hardware_interface/EffortJointInterface</hardwareInterface>
-      <mechanicalReduction>1</mechanicalReduction>
-    </actuator>
-  </transmission>
+  <xacro:SimpleTransmission n="1" joint="joint1" />
   <!--  Link 2 -->
   <link name="link2">
@@ -100,14 +104,5 @@
   </joint>
   <!-- Transmission 2 -->
-  <transmission name="tran2">
-    <type>transmission_interface/SimpleTransmission</type>
-    <joint name="joint2">
-      <hardwareInterface>hardware_interface/EffortJointInterface</hardwareInterface>
-    </joint>
-    <actuator name="motor2">
-      <hardwareInterface>hardware_interface/EffortJointInterface</hardwareInterface>
-      <mechanicalReduction>1</mechanicalReduction>
-    </actuator>
-  </transmission>
+  <xacro:SimpleTransmission n="2" joint="joint2" />
   <!--  Link 3 -->
   <link name="link3">
@@ -149,14 +144,5 @@
   </joint>
   <!-- Transmission 3 -->
-  <transmission name="tran3">
-    <type>transmission_interface/SimpleTransmission</type>
-    <joint name="joint3">
-      <hardwareInterface>hardware_interface/EffortJointInterface</hardwareInterface>
-    </joint>
-    <actuator name="motor3">
-      <hardwareInterface>hardware_interface/EffortJointInterface</hardwareInterface>
-      <mechanicalReduction>1</mechanicalReduction>
-    </actuator>
-  </transmission>
+  <xacro:SimpleTransmission n="3" joint="joint3" />
   <!--  Link 4 -->
   <link name="link4">
@@ -198,14 +184,5 @@
   </joint>
   <!-- Transmission 4 -->
-  <transmission name="tran4">
-    <type>transmission_interface/SimpleTransmission</type>
-    <joint name="joint4">
-      <hardwareInterface>hardware_interface/EffortJointInterface</hardwareInterface>
-    </joint>
-    <actuator name="motor4">
-      <hardwareInterface>hardware_interface/EffortJointInterface</hardwareInterface>
-      <mechanicalReduction>1</mechanicalReduction>
-    </actuator>
-  </transmission>
+  <xacro:SimpleTransmission n="4" joint="joint4" />
   <!--  Link 5 -->
   <link name="link5">
@@ -277,14 +254,5 @@
   </joint>
   <!-- Transmission 5 -->
-  <transmission name="tran5">
-    <type>transmission_interface/SimpleTransmission</type>
-    <joint name="grip_joint">
-      <hardwareInterface>hardware_interface/EffortJointInterface</hardwareInterface>
-    </joint>
-    <actuator name="motor7">
-      <hardwareInterface>hardware_interface/EffortJointInterface</hardwareInterface>
-      <mechanicalReduction>1</mechanicalReduction>
-    </actuator>
-  </transmission>
+  <xacro:SimpleTransmission n="5" joint="grip_joint" />
   <!--  Grip link sub -->
   <link name="grip_link_sub">
@@ -326,13 +294,4 @@
   </joint>
   <!-- Transmission 6 -->
-  <transmission name="tran6">
-    <type>transmission_interface/SimpleTransmission</type>
-    <joint name="grip_joint_sub">
-      <hardwareInterface>hardware_interface/EffortJointInterface</hardwareInterface>
-    </joint>
-    <actuator name="motor8">
-      <hardwareInterface>hardware_interface/EffortJointInterface</hardwareInterface>
-      <mechanicalReduction>1</mechanicalReduction>
-    </actuator>
-  </transmission>
+  <xacro:SimpleTransmission n="6" joint="grip_joint_sub" />
 </robot>

File: open_manipulator_with_tb3_description/urdf/open_manipulator_with_tb3_waffle_pi.urdf.xacro (robot description, xacro)
@@ -6,4 +6,17 @@
   <!-- Include OpenManipulator Chain Gazebo Parameter -->
   <xacro:include filename="$(find open_manipulator_with_tb3_description)/urdf/open_manipulator_with_tb3.gazebo.xacro" />
+  <!-- Transmission macro -->
+  <xacro:macro name="SimpleTransmission" params="joint n">
+    <transmission name="tran${n}">
+      <type>transmission_interface/SimpleTransmission</type>
+      <joint name="${joint}">
+	      <hardwareInterface>hardware_interface/PositionJointInterface</hardwareInterface>
+      </joint>
+      <actuator name="motor${n}">
+        <hardwareInterface>hardware_interface/PositionJointInterface</hardwareInterface>
+        <mechanicalReduction>1</mechanicalReduction>
+      </actuator>
+    </transmission>
+  </xacro:macro>
   <!-- Base fixed joint -->
   <joint name="base_fixed" type="fixed">
@@ -51,14 +64,5 @@
   </joint>
   <!-- Transmission 1 -->
-  <transmission name="tran1">
-    <type>transmission_interface/SimpleTransmission</type>
-    <joint name="joint1">
-      <hardwareInterface>hardware_interface/EffortJointInterface</hardwareInterface>
-    </joint>
-    <actuator name="motor1">
-      <hardwareInterface>hardware_interface/EffortJointInterface</hardwareInterface>
-      <mechanicalReduction>1</mechanicalReduction>
-    </actuator>
-  </transmission>
+  <xacro:SimpleTransmission n="1" joint="joint1" />
   <!--  Link 2 -->
   <link name="link2">
@@ -100,14 +104,5 @@
   </joint>
   <!-- Transmission 2 -->
-  <transmission name="tran2">
-    <type>transmission_interface/SimpleTransmission</type>
-    <joint name="joint2">
-      <hardwareInterface>hardware_interface/EffortJointInterface</hardwareInterface>
-    </joint>
-    <actuator name="motor2">
-      <hardwareInterface>hardware_interface/EffortJointInterface</hardwareInterface>
-      <mechanicalReduction>1</mechanicalReduction>
-    </actuator>
-  </transmission>
+  <xacro:SimpleTransmission n="2" joint="joint2" />
   <!--  Link 3 -->
   <link name="link3">
@@ -149,14 +144,5 @@
   </joint>
   <!-- Transmission 3 -->
-  <transmission name="tran3">
-    <type>transmission_interface/SimpleTransmission</type>
-    <joint name="joint3">
-      <hardwareInterface>hardware_interface/EffortJointInterface</hardwareInterface>
-    </joint>
-    <actuator name="motor3">
-      <hardwareInterface>hardware_interface/EffortJointInterface</hardwareInterface>
-      <mechanicalReduction>1</mechanicalReduction>
-    </actuator>
-  </transmission>
+  <xacro:SimpleTransmission n="3" joint="joint3" />
   <!--  Link 4 -->
   <link name="link4">
@@ -198,14 +184,5 @@
   </joint>
   <!-- Transmission 4 -->
-  <transmission name="tran4">
-    <type>transmission_interface/SimpleTransmission</type>
-    <joint name="joint4">
-      <hardwareInterface>hardware_interface/EffortJointInterface</hardwareInterface>
-    </joint>
-    <actuator name="motor4">
-      <hardwareInterface>hardware_interface/EffortJointInterface</hardwareInterface>
-      <mechanicalReduction>1</mechanicalReduction>
-    </actuator>
-  </transmission>
+  <xacro:SimpleTransmission n="4" joint="joint4" />
   <!--  Link 5 -->
   <link name="link5">
@@ -277,14 +254,5 @@
   </joint>
   <!-- Transmission 5 -->
-  <transmission name="tran5">
-    <type>transmission_interface/SimpleTransmission</type>
-    <joint name="grip_joint">
-      <hardwareInterface>hardware_interface/EffortJointInterface</hardwareInterface>
-    </joint>
-    <actuator name="motor7">
-      <hardwareInterface>hardware_interface/EffortJointInterface</hardwareInterface>
-      <mechanicalReduction>1</mechanicalReduction>
-    </actuator>
-  </transmission>
+  <xacro:SimpleTransmission n="5" joint="grip_joint" />
   <!--  Grip link sub -->
   <link name="grip_link_sub">
@@ -326,13 +294,4 @@
   </joint>
   <!-- Transmission 6 -->
-  <transmission name="tran6">
-    <type>transmission_interface/SimpleTransmission</type>
-    <joint name="grip_joint_sub">
-      <hardwareInterface>hardware_interface/EffortJointInterface</hardwareInterface>
-    </joint>
-    <actuator name="motor8">
-      <hardwareInterface>hardware_interface/EffortJointInterface</hardwareInterface>
-      <mechanicalReduction>1</mechanicalReduction>
-    </actuator>
-  </transmission>
+  <xacro:SimpleTransmission n="6" joint="grip_joint_sub" />
 </robot>
