Commit message: changed gripper position -> effort controller

File: turtlebot3_manipulation_description/urdf/open_manipulator_x.transmission.xacro (robot description, xacro)
@@ -2,5 +2,5 @@
 <robot xmlns:xacro="http://ros.org/wiki/xacro">
   <!-- Transmission macro -->
-  <xacro:macro name="SimpleTransmission" params="joint n">
+  <xacro:macro name="SimpleTransmissionPosition" params="joint n">
     <transmission name="tran${n}">
       <type>transmission_interface/SimpleTransmission</type>
@@ -14,15 +14,28 @@
     </transmission>
   </xacro:macro>
+  <!-- Transmission macro -->
+  <xacro:macro name="SimpleTransmissionEffort" params="joint n">
+    <transmission name="tran${n}">
+      <type>transmission_interface/SimpleTransmission</type>
+      <joint name="${joint}">
+        <hardwareInterface>hardware_interface/EffortJointInterface</hardwareInterface>
+      </joint>
+      <actuator name="motor${n}">
+        <hardwareInterface>hardware_interface/EffortJointInterface</hardwareInterface>
+        <mechanicalReduction>1</mechanicalReduction>
+      </actuator>
+    </transmission>
+  </xacro:macro>
   <!-- Transmission 1 -->
-  <xacro:SimpleTransmission n="1" joint="joint1" />
+  <xacro:SimpleTransmissionPosition n="1" joint="joint1" />
   <!-- Transmission 2 -->
-  <xacro:SimpleTransmission n="2" joint="joint2" />
+  <xacro:SimpleTransmissionPosition n="2" joint="joint2" />
   <!-- Transmission 3 -->
-  <xacro:SimpleTransmission n="3" joint="joint3" />
+  <xacro:SimpleTransmissionPosition n="3" joint="joint3" />
   <!-- Transmission 4 -->
-  <xacro:SimpleTransmission n="4" joint="joint4" />
+  <xacro:SimpleTransmissionPosition n="4" joint="joint4" />
   <!-- Transmission 5 -->
-  <xacro:SimpleTransmission n="5" joint="gripper" />
+  <xacro:SimpleTransmissionEffort n="5" joint="gripper" />
   <!-- Transmission 6 -->
-  <xacro:SimpleTransmission n="6" joint="gripper_sub" />
+  <xacro:SimpleTransmissionEffort n="6" joint="gripper_sub" />
 </robot>
