Commit message: fixed wheel slip bug

File: turtlebot3_manipulation_description/urdf/open_manipulator_x.gazebo.xacro (robot description, xacro)
@@ -36,4 +36,5 @@
       <controlPeriod>0.001</controlPeriod>
       <robotSimType>gazebo_ros_control/DefaultRobotHWSim</robotSimType>
+      <legacyModeNS>true</legacyModeNS>
     </plugin>
   </gazebo>
@@ -45,4 +46,5 @@
       <multiplier>1.0</multiplier>
       <offset>0.0</offset>
+      <hasPID>/gazebo_ros_control/pid_gains/gripper_sub</hasPID>
     </plugin>
   </gazebo>

File: turtlebot3_manipulation_description/urdf/open_manipulator_x.urdf.xacro (robot description, xacro)
@@ -146,8 +146,12 @@
     <inertial>
       <origin xyz="4.4206755e-02 3.6839985e-07 8.9142216e-03" />
-      <mass value="1.4327573e-01" />
+      <!-- <mass value="1.4327573e-01" />
       <inertia ixx="8.0870749e-05" ixy="0.0" ixz="-1.0157896e-06"
                iyy="7.5980465e-05" iyz="0.0"
-               izz="9.3127351e-05" />
+               izz="9.3127351e-05" /> -->
+      <mass value="1.0e-03" />
+      <inertia ixx="1.0e-03" ixy="0.0" ixz="0.0"
+               iyy="1.0e-03" iyz="0.0"
+               izz="1.0e-03" />
     </inertial>
   </link>
