Commit message: add mesh files
Signed-off-by: Hye-jong KIM <hjkim@robotis.com>

File: turtlebot3_manipulation_description/urdf/turtlebot3_manipulation.urdf.xacro (robot description, xacro)
@@ -2,10 +2,4 @@
 <!-- TurtleBot3 Manipulation -->
 <robot name="turtlebot3_manipulation" xmlns:xacro="http://ros.org/wiki/xacro">
-  <!-- Include TurtleBot3 Waffle Pi URDF -->
-  <!-- <xacro:include filename="$(find turtlebot3_description)/urdf/turtlebot3_waffle_pi.urdf" /> -->
-  <!-- Include TurtleBot3 OpenManipulatorX URDF -->
-  <!-- <xacro:include filename="$(find open_manipulator_x_description)/urdf/open_manipulator_x.urdf.xacro" /> -->
-  <!-- Include OpenManipulator Chain Gazebo Parameter -->
-  <!-- <xacro:include filename="$(find turtlebot3_description)/urdf/turtlebot3_description.gazebo.xacro" /> -->
   <!-- Transmission macro -->
   <xacro:macro name="SimpleTransmission" params="joint n">
@@ -63,5 +57,5 @@
       <origin xyz="-0.064 0 0.0" rpy="0 0 0"/>
       <geometry>
-        <mesh filename="package://turtlebot3_description/meshes/bases/waffle_pi_base.stl" scale="0.001 0.001 0.001"/>
+        <mesh filename="package://turtlebot3_manipulation_description/meshes/bases/waffle_pi_base.stl" scale="0.001 0.001 0.001"/>
       </geometry>
       <material name="light_black"/>
@@ -91,5 +85,5 @@
       <origin xyz="0 0 0" rpy="1.57 0 0"/>
       <geometry>
-        <mesh filename="package://turtlebot3_description/meshes/wheels/left_tire.stl" scale="0.001 0.001 0.001"/>
+        <mesh filename="package://turtlebot3_manipulation_description/meshes/wheels/left_tire.stl" scale="0.001 0.001 0.001"/>
       </geometry>
       <material name="dark"/>
@@ -119,5 +113,5 @@
       <origin xyz="0 0 0" rpy="1.57 0 0"/>
       <geometry>
-        <mesh filename="package://turtlebot3_description/meshes/wheels/right_tire.stl" scale="0.001 0.001 0.001"/>
+        <mesh filename="package://turtlebot3_manipulation_description/meshes/wheels/right_tire.stl" scale="0.001 0.001 0.001"/>
       </geometry>
       <material name="dark"/>
@@ -192,5 +186,5 @@
       <origin xyz="0 0 0.0" rpy="0 0 0"/>
       <geometry>
-        <mesh filename="package://turtlebot3_description/meshes/sensors/lds.stl" scale="0.001 0.001 0.001"/>
+        <mesh filename="package://turtlebot3_manipulation_description/meshes/sensors/lds.stl" scale="0.001 0.001 0.001"/>
       </geometry>
       <material name="dark"/>
@@ -247,12 +241,12 @@
       <origin xyz="0 0 0" rpy="0 0 0"/>
       <geometry>
-        <mesh filename="package://open_manipulator_x_description/meshes/link1.stl" scale="0.001 0.001 0.001"/>
-      </geometry>
-      <material name="grey"/>
-    </visual>
-    <collision>
-      <origin xyz="0 0 0" rpy="0 0 0"/>
-      <geometry>
-        <mesh filename="package://open_manipulator_x_description/meshes/link1.stl" scale="0.001 0.001 0.001"/>
+        <mesh filename="package://turtlebot3_manipulation_description/meshes/manipulator/link1.stl" scale="0.001 0.001 0.001"/>
+      </geometry>
+      <material name="grey"/>
+    </visual>
+    <collision>
+      <origin xyz="0 0 0" rpy="0 0 0"/>
+      <geometry>
+        <mesh filename="package://turtlebot3_manipulation_description/meshes/manipulator/link1.stl" scale="0.001 0.001 0.001"/>
       </geometry>
     </collision>
@@ -287,5 +281,5 @@
       <origin xyz="0 0 0.019" rpy="0 0 0"/>
       <geometry>
-        <mesh filename="package://open_manipulator_x_description/meshes/link2.stl" scale="0.001 0.001 0.001"/>
+        <mesh filename="package://turtlebot3_manipulation_description/meshes/manipulator/link2.stl" scale="0.001 0.001 0.001"/>
       </geometry>
       <material name="grey"/>
@@ -294,5 +288,5 @@
       <origin xyz="0 0 0.019" rpy="0 0 0"/>
       <geometry>
-        <mesh filename="package://open_manipulator_x_description/meshes/link2.stl" scale="0.001 0.001 0.001"/>
+        <mesh filename="package://turtlebot3_manipulation_description/meshes/manipulator/link2.stl" scale="0.001 0.001 0.001"/>
       </geometry>
     </collision>
@@ -327,12 +321,12 @@
       <origin xyz="0 0 0" rpy="0 0 0"/>
       <geometry>
-        <mesh filename="package://open_manipulator_x_description/meshes/link3.stl" scale="0.001 0.001 0.001"/>
-      </geometry>
-      <material name="grey"/>
-    </visual>
-    <collision>
-      <origin xyz="0 0 0" rpy="0 0 0"/>
-      <geometry>
-        <mesh filename="package://open_manipulator_x_description/meshes/link3.stl" scale="0.001 0.001 0.001"/>
+        <mesh filename="package://turtlebot3_manipulation_description/meshes/manipulator/link3.stl" scale="0.001 0.001 0.001"/>
+      </geometry>
+      <material name="grey"/>
+    </visual>
+    <collision>
+      <origin xyz="0 0 0" rpy="0 0 0"/>
+      <geometry>
+        <mesh filename="package://turtlebot3_manipulation_description/meshes/manipulator/link3.stl" scale="0.001 0.001 0.001"/>
       </geometry>
     </collision>
@@ -367,12 +361,12 @@
       <origin xyz="0 0 0" rpy="0 0 0"/>
       <geometry>
-        <mesh filename="package://open_manipulator_x_description/meshes/link4.stl" scale="0.001 0.001 0.001"/>
-      </geometry>
-      <material name="grey"/>
-    </visual>
-    <collision>
-      <origin xyz="0 0 0" rpy="0 0 0"/>
-      <geometry>
-        <mesh filename="package://open_manipulator_x_description/meshes/link4.stl" scale="0.001 0.001 0.001"/>
+        <mesh filename="package://turtlebot3_manipulation_description/meshes/manipulator/link4.stl" scale="0.001 0.001 0.001"/>
+      </geometry>
+      <material name="grey"/>
+    </visual>
+    <collision>
+      <origin xyz="0 0 0" rpy="0 0 0"/>
+      <geometry>
+        <mesh filename="package://turtlebot3_manipulation_description/meshes/manipulator/link4.stl" scale="0.001 0.001 0.001"/>
       </geometry>
     </collision>
@@ -407,12 +401,12 @@
       <origin xyz="0 0 0" rpy="0 0 0"/>
       <geometry>
-        <mesh filename="package://open_manipulator_x_description/meshes/link5.stl" scale="0.001 0.001 0.001"/>
-      </geometry>
-      <material name="grey"/>
-    </visual>
-    <collision>
-      <origin xyz="0 0 0" rpy="0 0 0"/>
-      <geometry>
-        <mesh filename="package://open_manipulator_x_description/meshes/link5.stl" scale="0.001 0.001 0.001"/>
+        <mesh filename="package://turtlebot3_manipulation_description/meshes/manipulator/link5.stl" scale="0.001 0.001 0.001"/>
+      </geometry>
+      <material name="grey"/>
+    </visual>
+    <collision>
+      <origin xyz="0 0 0" rpy="0 0 0"/>
+      <geometry>
+        <mesh filename="package://turtlebot3_manipulation_description/meshes/manipulator/link5.stl" scale="0.001 0.001 0.001"/>
       </geometry>
     </collision>
@@ -437,5 +431,5 @@
       <origin xyz="0.0 0.0 0" rpy="0 0 0"/>
       <geometry>
-        <mesh filename="package://open_manipulator_x_description/meshes/link_grip_l.stl" scale="0.001 0.001 0.001"/>
+        <mesh filename="package://turtlebot3_manipulation_description/meshes/manipulator/link_grip_l.stl" scale="0.001 0.001 0.001"/>
       </geometry>
       <material name="grey"/>
@@ -444,5 +438,5 @@
       <origin xyz="0.0 0.0 0" rpy="0 0 0"/>
       <geometry>
-        <mesh filename="package://open_manipulator_x_description/meshes/link_grip_l.stl" scale="0.001 0.001 0.001"/>
+        <mesh filename="package://turtlebot3_manipulation_description/meshes/manipulator/link_grip_l.stl" scale="0.001 0.001 0.001"/>
       </geometry>
     </collision>
@@ -477,5 +471,5 @@
       <origin xyz="0.0 -0.0 0" rpy="0 0 0"/>
       <geometry>
-        <mesh filename="package://open_manipulator_x_description/meshes/link_grip_r.stl" scale="0.001 0.001 0.001"/>
+        <mesh filename="package://turtlebot3_manipulation_description/meshes/manipulator/link_grip_r.stl" scale="0.001 0.001 0.001"/>
       </geometry>
       <material name="grey"/>
@@ -484,5 +478,5 @@
       <origin xyz="0.0 -0.0 0" rpy="0 0 0"/>
       <geometry>
-        <mesh filename="package://open_manipulator_x_description/meshes/link_grip_r.stl" scale="0.001 0.001 0.001"/>
+        <mesh filename="package://turtlebot3_manipulation_description/meshes/manipulator/link_grip_r.stl" scale="0.001 0.001 0.001"/>
       </geometry>
     </collision>

Commit message: fix urdf
Signed-off-by: Hye-jong KIM <hjkim@robotis.com>

File: turtlebot3_manipulation_description/urdf/turtlebot3_manipulation.urdf.xacro (robot description, xacro)
@@ -180,5 +180,5 @@
     <parent link="base_link"/>
     <child link="base_scan"/>
-    <origin xyz="-0.064 0 0.122" rpy="0 0 0"/>
+    <origin xyz="-0.024 0 0.122" rpy="0 0 0"/>
   </joint>
   <link name="base_scan">
@@ -234,5 +234,5 @@
     <parent link="base_link"/>
     <child link="link1"/>
-    <origin xyz="-0.136 0.0 0.090" rpy="0 0 0"/>
+    <origin xyz="-0.092 0.0 0.091" rpy="0 0 0"/>
   </joint>
   <!-- Link 1 -->
@@ -246,16 +246,9 @@
     </visual>
     <collision>
-      <origin xyz="0 0 0" rpy="0 0 0"/>
-      <geometry>
-        <mesh filename="package://turtlebot3_manipulation_description/meshes/manipulator/link1.stl" scale="0.001 0.001 0.001"/>
-      </geometry>
-    </collision>
-<!--    <inertial>
-      <origin xyz="0 0 0" />
-      <mass value="0.082" />
-      <inertia ixx="0.1" ixy="0.0" ixz="0.0"
-               iyy="0.1" iyz="0.0"
-               izz="0.1" />
-    </inertial>-->
+      <origin xyz="0.0 0 0.017" rpy="0 0 0"/>
+      <geometry>
+        <box size="0.0465 0.0285 0.034"/>
+      </geometry>
+    </collision>
      <inertial>
       <origin xyz="3.0876154e-04 0.0000000e+00 -1.2176461e-04" />
@@ -286,16 +279,9 @@
     </visual>
     <collision>
-      <origin xyz="0 0 0.019" rpy="0 0 0"/>
-      <geometry>
-        <mesh filename="package://turtlebot3_manipulation_description/meshes/manipulator/link2.stl" scale="0.001 0.001 0.001"/>
-      </geometry>
-    </collision>
-<!--    <inertial>
-      <origin xyz="0 0 0" />
-      <mass value="0.098" />
-      <inertia ixx="0.1" ixy="0.0" ixz="0.0"
-               iyy="0.1" iyz="0.0"
-               izz="0.1" />
-    </inertial>-->
+      <origin xyz="0 0 0.0475" rpy="0 0 0"/>
+      <geometry>
+        <box size="0.034 0.0285 0.0465"/>
+      </geometry>
+    </collision>
      <inertial>
       <origin xyz="-3.0184870e-04 5.4043684e-04 0.047433464" />
