Commit message: URDF update
Signed-off-by: Hye-jong KIM <hjkim@robotis.com>

File: turtlebot3_manipulation_description/urdf/turtlebot3_manipulation.urdf.xacro (robot description, xacro)
@@ -345,7 +345,7 @@
     </visual>
     <collision>
-      <origin xyz="0.08765 0 0" rpy="0 0 0"/>
-      <geometry>
-        <box size="0.11485 0.034 0.02375"/>
+      <origin xyz="0.0675 0 0" rpy="0 0 0"/>
+      <geometry>
+        <box size="0.135 0.034 0.02375"/>
       </geometry>
     </collision>
@@ -378,5 +378,5 @@
     </visual>
     <collision>
-      <origin xyz="0.0555 0 0.0705" rpy="0 0 0"/>
+      <origin xyz="0.0555 0 0.00705" rpy="0 0 0"/>
       <geometry>
         <box size="0.055 0.130 0.061"/>
