Commit message: add joint damping in urdf
Signed-off-by: Hye-jong KIM <hjkim@robotis.com>

File: turtlebot3_manipulation_description/urdf/open_manipulator_x.urdf.xacro (robot description, xacro)
@@ -40,4 +40,5 @@
       <axis xyz="0 0 1"/>
       <limit velocity="4.8" effort="1" lower="${-pi*0.9}" upper="${pi*0.9}" />
+      <dynamics damping="0.1"/>
     </joint>
     <link name="${prefix}link2">
@@ -71,4 +72,5 @@
       <axis xyz="0 1 0"/>
       <limit velocity="4.8" effort="1" lower="${-pi*0.57}" upper="${pi*0.5}" />
+      <dynamics damping="0.1"/>
     </joint>
     <link name="${prefix}link3">
@@ -102,4 +104,5 @@
       <axis xyz="0 1 0"/>
       <limit velocity="4.8" effort="1" lower="${-pi*0.3}" upper="${pi*0.44}" />
+      <dynamics damping="0.1"/>
     </joint>
     <link name="${prefix}link4">
@@ -133,4 +136,5 @@
       <axis xyz="0 1 0"/>
       <limit velocity="4.8" effort="1" lower="${-pi*0.57}" upper="${pi*0.65}" />
+      <dynamics damping="0.1"/>
     </joint>
     <link name="${prefix}link5">
@@ -164,4 +168,5 @@
       <axis xyz="0 1 0"/>
       <limit velocity="4.8" effort="1" lower="-0.010" upper="0.019" />
+      <dynamics damping="0.1"/>
     </joint>
     <link name="${prefix}gripper_left_link">
@@ -196,4 +201,5 @@
       <limit velocity="4.8" effort="1" lower="-0.010" upper="0.019" />
       <mimic joint="${prefix}gripper_left_joint" multiplier="1"/>
+      <dynamics damping="0.1"/>
     </joint>
     <link name="${prefix}gripper_right_link">

Commit message: Modified gripper position limit
Signed-off-by: Darby Lim <thlim@robotis.com>

File: turtlebot3_manipulation_description/urdf/open_manipulator_x.urdf.xacro (robot description, xacro)
@@ -158,5 +158,5 @@
     <origin xyz="0.0817 0.021 0.0" rpy="0 0 0"/>
     <axis xyz="0 1 0"/>
-    <limit velocity="4.8" effort="1" lower="-0.010" upper="0.019" />
+    <limit velocity="4.8" effort="1" lower="-0.010" upper="0.010" />
   </joint>
   <link name="${prefix}gripper_left_link">
@@ -188,5 +188,5 @@
     <origin xyz="0.0817 -0.021 0" rpy="0 0 0"/>
     <axis xyz="0 -1 0"/>
-    <limit velocity="4.8" effort="1" lower="-0.010" upper="0.019" />
+    <limit velocity="4.8" effort="1" lower="-0.010" upper="0.010" />
     <mimic joint="${prefix}gripper_left_joint" multiplier="1"/>
   </joint>

Commit message: Deleted unused codes
Signed-off-by: Darby Lim <thlim@robotis.com>

File: turtlebot3_manipulation_description/urdf/open_manipulator_x.urdf.xacro (robot description, xacro)
@@ -19,8 +19,6 @@
       </visual>
       <collision>
-  <!--      <origin xyz="0 0 0.017" rpy="0 0 0"/>-->
-        <origin xyz="0 0 0" rpy="0 0 0"/>
-        <geometry>
-  <!--        <box size="0.0465 0.0285 0.024"/>-->
+        <origin xyz="0 0 0" rpy="0 0 0"/>
+        <geometry>
           <mesh filename="${meshes_file_direction}/link1.stl" scale="0.001 0.001 0.001"/>
         </geometry>
@@ -51,8 +49,6 @@
       </visual>
       <collision>
-  <!--      <origin xyz="0 0 0.0475" rpy="0 0 0"/>-->
         <origin xyz="0 0 0.019" rpy="0 0 0"/>
         <geometry>
-  <!--        <box size="0.0285 0.034 0.0465"/>-->
           <mesh filename="${meshes_file_direction}/link2.stl" scale="0.001 0.001 0.001"/>
         </geometry>
@@ -83,8 +79,6 @@
       </visual>
       <collision>
-  <!--      <origin xyz="0 0 0.09265" rpy="0 0 0"/>-->
-        <origin xyz="0 0 0" rpy="0 0 0"/>
-        <geometry>
-  <!--        <box size="0.02375 0.034 0.12485"/>-->
+        <origin xyz="0 0 0" rpy="0 0 0"/>
+        <geometry>
           <mesh filename="${meshes_file_direction}/link3.stl" scale="0.001 0.001 0.001"/>
         </geometry>
@@ -115,8 +109,6 @@
       </visual>
       <collision>
-  <!--      <origin xyz="0.0675 0 0" rpy="0 0 0"/>-->
-        <origin xyz="0 0 0" rpy="0 0 0"/>
-        <geometry>
-  <!--        <box size="0.135 0.034 0.02375"/>-->
+        <origin xyz="0 0 0" rpy="0 0 0"/>
+        <geometry>
           <mesh filename="${meshes_file_direction}/link4.stl" scale="0.001 0.001 0.001"/>
         </geometry>
@@ -147,8 +139,6 @@
       </visual>
       <collision>
-  <!--      <origin xyz="0.0555 0 0.00705" rpy="0 0 0"/>-->
-        <origin xyz="0 0 0" rpy="0 0 0"/>
-        <geometry>
-  <!--        <box size="0.055 0.130 0.061"/>-->
+        <origin xyz="0 0 0" rpy="0 0 0"/>
+        <geometry>
           <mesh filename="${meshes_file_direction}/link5.stl" scale="0.001 0.001 0.001"/>
         </geometry>
@@ -179,8 +169,6 @@
       </visual>
       <collision>
-  <!--      <origin xyz="0.052 0.0075 0" rpy="0 0 0"/>-->
-        <origin xyz="0 0 0" rpy="0 0 0"/>
-        <geometry>
-  <!--        <box size="0.070 0.035 0.055"/>-->
+        <origin xyz="0 0 0" rpy="0 0 0"/>
+        <geometry>
           <mesh filename="${meshes_file_direction}/gripper_left_palm.stl" scale="0.001 0.001 0.001"/>
         </geometry>
@@ -212,8 +200,6 @@
       </visual>
       <collision>
-  <!--      <origin xyz="0.052 -0.0075 0" rpy="0 0 0"/>-->
-        <origin xyz="0 0 0" rpy="0 0 0"/>
-        <geometry>
-  <!--        <box size="0.070 0.035 0.055"/>-->
+        <origin xyz="0 0 0" rpy="0 0 0"/>
+        <geometry>
           <mesh filename="${meshes_file_direction}/gripper_right_palm.stl" scale="0.001 0.001 0.001"/>
         </geometry>
@@ -240,11 +226,4 @@
         <material name="red"/>
        </visual>
-  <!--    <inertial>
-        <origin xyz="0 0 0" />
-        <mass value="1.0e-04" />
-        <inertia ixx="1.0e-04" ixy="0.0" ixz="0.0"
-                 iyy="1.0e-04" iyz="0.0"
-                 izz="1.0e-04" />
-      </inertial>-->
     </link>
   </xacro:macro>

Commit message: modified teleop and added an example

File: turtlebot3_manipulation_description/urdf/open_manipulator_x.urdf.xacro (robot description, xacro)
@@ -182,4 +182,9 @@
       </inertial>
     </link>
+    <joint name="${prefix}gripper_right_joint_mimic" type="fixed">
+      <parent link="${prefix}link5" />
+      <child link="dummy_mimic_fix" />
+    </joint>
+    <link name="dummy_mimic_fix"/>
     <joint name="${prefix}gripper_right_joint" type="prismatic">
       <parent link="${prefix}link5"/>

Commit message: converted stl collision to box collision

File: turtlebot3_manipulation_description/urdf/open_manipulator_x.urdf.xacro (robot description, xacro)
@@ -21,5 +21,5 @@
         <origin xyz="0 0 0" rpy="0 0 0"/>
         <geometry>
-          <mesh filename="${meshes_file_direction}/link1.stl" scale="0.001 0.001 0.001"/>
+          <box size="0.05 0.05 0.05"/>
         </geometry>
       </collision>
