Commit message: Modified gripper names
Signed-off-by: Darby Lim <thlim@robotis.com>

File: turtlebot3_manipulation_description/gazebo/open_manipulator_x.gazebo.xacro (robot description, xacro)
@@ -22,6 +22,6 @@
   <xacro:Link reference="${prefix}link4"/>
   <xacro:Link reference="${prefix}link5"/>
-  <xacro:Link reference="${prefix}gripper_link"/>
-  <xacro:Link reference="${prefix}gripper_link_sub"/>
+  <xacro:Link reference="${prefix}gripper_left_link"/>
+  <xacro:Link reference="${prefix}gripper_right_link"/>
   <gazebo reference="${prefix}end_effector_link">
     <material>Gazebo/Red</material>

File: turtlebot3_manipulation_description/urdf/open_manipulator_x.urdf.xacro (robot description, xacro)
@@ -22,4 +22,5 @@
       <geometry>
         <box size="0.0465 0.0285 0.034"/>
+        <!-- <mesh filename="${meshes_file_direction}/link1.stl" scale="0.001 0.001 0.001"/> -->
       </geometry>
     </collision>
@@ -51,4 +52,5 @@
       <geometry>
         <box size="0.0285 0.034 0.0465"/>
+        <!-- <mesh filename="${meshes_file_direction}/link2.stl" scale="0.001 0.001 0.001"/> -->
       </geometry>
     </collision>
@@ -80,4 +82,5 @@
       <geometry>
         <box size="0.02375 0.034 0.12485"/>
+        <!-- <mesh filename="${meshes_file_direction}/link3.stl" scale="0.001 0.001 0.001"/> -->
       </geometry>
     </collision>
@@ -109,4 +112,5 @@
       <geometry>
         <box size="0.135 0.034 0.02375"/>
+        <!-- <mesh filename="${meshes_file_direction}/link4.stl" scale="0.001 0.001 0.001"/> -->
       </geometry>
     </collision>
@@ -138,4 +142,5 @@
       <geometry>
         <box size="0.055 0.130 0.061"/>
+        <!-- <mesh filename="${meshes_file_direction}/link5.stl" scale="0.001 0.001 0.001"/> -->
       </geometry>
     </collision>
@@ -148,5 +153,12 @@
     </inertial>
   </link>
-  <link name="${prefix}gripper_link">
+  <joint name="${prefix}gripper_left_joint" type="prismatic">
+    <parent link="${prefix}link5"/>
+    <child link="${prefix}gripper_left_link"/>
+    <origin xyz="0.0817 0.021 0.0" rpy="0 0 0"/>
+    <axis xyz="0 1 0"/>
+    <limit velocity="4.8" effort="1" lower="-0.010" upper="0.019" />
+  </joint>
+  <link name="${prefix}gripper_left_link">
     <visual>
       <origin xyz="0.0 0.0 0" rpy="0 0 0"/>
@@ -160,4 +172,5 @@
       <geometry>
         <box size="0.070 0.035 0.055"/>
+        <!-- <mesh filename="${meshes_file_direction}/gripper_left_palm.stl" scale="0.001 0.001 0.001"/> -->
       </geometry>
     </collision>
@@ -170,12 +183,13 @@
     </inertial>
   </link>
-  <joint name="${prefix}gripper" type="prismatic">
+  <joint name="${prefix}gripper_right_joint" type="prismatic">
     <parent link="${prefix}link5"/>
-    <child link="${prefix}gripper_link"/>
-    <origin xyz="0.0817 0.021 0.0" rpy="0 0 0"/>
-    <axis xyz="0 1 0"/>
+    <child link="${prefix}gripper_right_link"/>
+    <origin xyz="0.0817 -0.021 0" rpy="0 0 0"/>
+    <axis xyz="0 -1 0"/>
     <limit velocity="4.8" effort="1" lower="-0.010" upper="0.019" />
-  </joint>
-  <link name="${prefix}gripper_link_sub">
+    <mimic joint="${prefix}gripper" multiplier="1"/>
+  </joint>
+  <link name="${prefix}gripper_right_link">
     <visual>
       <origin xyz="0.0 -0.0 0" rpy="0 0 0"/>
@@ -189,4 +203,5 @@
       <geometry>
         <box size="0.070 0.035 0.055"/>
+        <!-- <mesh filename="${meshes_file_direction}/gripper_right_palm.stl" scale="0.001 0.001 0.001"/> -->
       </geometry>
     </collision>
@@ -199,12 +214,4 @@
     </inertial>
   </link>
-  <joint name="${prefix}gripper_sub" type="prismatic">
-    <parent link="${prefix}link5"/>
-    <child link="${prefix}gripper_link_sub"/>
-    <origin xyz="0.0817 -0.021 0" rpy="0 0 0"/>
-    <axis xyz="0 -1 0"/>
-    <limit velocity="4.8" effort="1" lower="-0.010" upper="0.019" />
-    <mimic joint="${prefix}gripper" multiplier="1"/>
-  </joint>
   <joint name="${prefix}end_effector_joint" type="fixed">
     <parent link="${prefix}link5"/>

Commit message: Added transmission tags
Signed-off-by: Darby Lim <thlim@robotis.com>

File: turtlebot3_manipulation_description/gazebo/open_manipulator_x.gazebo.xacro (robot description, xacro)
@@ -6,4 +6,16 @@
 <robot xmlns:xacro="http://ros.org/wiki/xacro">
   <xacro:macro name="open_manipulator_x_gazebo" params="prefix">
+  <xacro:macro name="SimpleTransmission" params="trans joint actuator">
+    <transmission name="${trans}">
+      <type>transmission_interface/SimpleTransmission</type>
+      <joint name="${joint}">
+        <hardwareInterface>PositionJointInterface</hardwareInterface>
+      </joint>
+      <actuator name="${actuator}">
+        <mechanicalReduction>1</mechanicalReduction>
+        <hardwareInterface>PositionJointInterface</hardwareInterface>
+      </actuator>
+    </transmission>
+  </xacro:macro>
   <xacro:macro name="Link" params="reference">
     <gazebo reference="${reference}">
@@ -27,4 +39,10 @@
     <material>Gazebo/Red</material>
   </gazebo>
+  <xacro:SimpleTransmission trans="${prefix}trans1" joint="${prefix}joint1" actuator="${prefix}actuator1" />
+  <xacro:SimpleTransmission trans="${prefix}trans2" joint="${prefix}joint2" actuator="${prefix}actuator2" />
+  <xacro:SimpleTransmission trans="${prefix}trans3" joint="${prefix}joint3" actuator="${prefix}actuator3" />
+  <xacro:SimpleTransmission trans="${prefix}trans4" joint="${prefix}joint4" actuator="${prefix}actuator4" />
+  <xacro:SimpleTransmission trans="${prefix}trans5" joint="${prefix}gripper_left_joint" actuator="${prefix}actuator5" />
+  <xacro:SimpleTransmission trans="${prefix}trans6" joint="${prefix}gripper_right_joint" actuator="${prefix}actuator6" />
   </xacro:macro>
 </robot>
