Commit message: Deleted imu gazebo plugin
Signed-off-by: Darby Lim <thlim@robotis.com>

File: turtlebot3_manipulation_description/gazebo/turtlebot3_waffle_pi.gazebo.xacro (robot description, xacro)
@@ -51,35 +51,10 @@
   </gazebo>
   <gazebo reference="${prefix}imu_link">
+    <material>Gazebo/Grey</material>
     <sensor type="imu" name="imu">
       <always_on>true</always_on>
+      <update_rate>100.0</update_rate>
       <visualize>${imu_visual}</visualize>
     </sensor>
-    <material>Gazebo/Grey</material>
-    <plugin name="imu_plugin" filename="libgazebo_ros_imu.so">
-      <alwaysOn>true</alwaysOn>
-      <bodyName>imu_link</bodyName>
-      <frameName>imu_link</frameName>
-      <topicName>imu</topicName>
-      <serviceName>imu_service</serviceName>
-      <gaussianNoise>0.0</gaussianNoise>
-      <updateRate>0</updateRate>
-      <imu>
-        <noise>
-          <type>gaussian</type>
-          <rate>
-            <mean>0.0</mean>
-            <stddev>2e-4</stddev>
-            <bias_mean>0.0000075</bias_mean>
-            <bias_stddev>0.0000008</bias_stddev>
-          </rate>
-          <accel>
-            <mean>0.0</mean>
-            <stddev>1.7e-2</stddev>
-            <bias_mean>0.1</bias_mean>
-            <bias_stddev>0.001</bias_stddev>
-          </accel>
-        </noise>
-      </imu>
-    </plugin>
   </gazebo>
   <gazebo reference="${prefix}base_scan">
