Commit message: Added sensor tag registering imu and modified gripper names
Signed-off-by: Darby Lim <thlim@robotis.com>

File: turtlebot3_manipulation_description/ros2_control/turtlebot3_manipulation_system.ros2_control.xacro (robot description, xacro)
@@ -41,4 +41,16 @@
         <state_interface name="velocity"/>
       </joint>
+      <sensor name="imu">
+        <state_interface name="orientation.x"/>
+        <state_interface name="orientation.y"/>
+        <state_interface name="orientation.z"/>
+        <state_interface name="orientation.w"/>
+        <state_interface name="angular_velocity.x"/>
+        <state_interface name="angular_velocity.y"/>
+        <state_interface name="angular_velocity.z"/>
+        <state_interface name="linear_acceleration.x"/>
+        <state_interface name="linear_acceleration.y"/>
+        <state_interface name="linear_acceleration.z"/>
+      </sensor>
       <joint name="${prefix}joint1">
         <command_interface name="position">
@@ -69,5 +81,5 @@
         <state_interface name="position"/>
       </joint>
-      <joint name="${prefix}gripper">
+      <joint name="${prefix}gripper_left_joint">
         <command_interface name="position">
           <param name="min">-0.010</param>
@@ -76,5 +88,7 @@
         <state_interface name="position"/>
       </joint>
-      <joint name="${prefix}gripper_sub">
+      <joint name="${prefix}gripper_right_joint">
+        <param name="mimic">gripper_left_joint</param>
+        <param name="multiplier">1</param>
         <command_interface name="position">
           <param name="min">-0.010</param>

Commit message: change controller name
Signed-off-by: Hye-jong KIM <hjkim@robotis.com>

File: turtlebot3_manipulation_description/ros2_control/turtlebot3_manipulation_system.ros2_control.xacro (robot description, xacro)
@@ -59,4 +59,5 @@
         </command_interface>
         <state_interface name="position"/>
+        <state_interface name="velocity"/>
       </joint>
       <joint name="${prefix}joint2">
@@ -66,4 +67,5 @@
         </command_interface>
         <state_interface name="position"/>
+        <state_interface name="velocity"/>
       </joint>
       <joint name="${prefix}joint3">
@@ -73,4 +75,5 @@
         </command_interface>
         <state_interface name="position"/>
+        <state_interface name="velocity"/>
       </joint>
       <joint name="${prefix}joint4">
@@ -80,4 +83,5 @@
         </command_interface>
         <state_interface name="position"/>
+        <state_interface name="velocity"/>
       </joint>
       <joint name="${prefix}gripper_left_joint">

File: turtlebot3_manipulation_description/urdf/open_manipulator_x.urdf.xacro (robot description, xacro)
@@ -177,8 +177,8 @@
     <inertial>
       <origin xyz="0 0 0" />
-      <mass value="1.0e-03" />
-      <inertia ixx="1.0e-03" ixy="0.0" ixz="0.0"
-               iyy="1.0e-03" iyz="0.0"
-               izz="1.0e-03" />
+      <mass value="1.0e-02" />
+      <inertia ixx="1.0e-06" ixy="0.0" ixz="0.0"
+               iyy="1.0e-06" iyz="0.0"
+               izz="1.0e-06" />
     </inertial>
   </link>
@@ -208,8 +208,8 @@
     <inertial>
       <origin xyz="0 0 0" />
-      <mass value="1.0e-03" />
-      <inertia ixx="1.0e-03" ixy="0.0" ixz="0.0"
-               iyy="1.0e-03" iyz="0.0"
-               izz="1.0e-03" />
+      <mass value="1.0e-02" />
+      <inertia ixx="1.0e-06" ixy="0.0" ixz="0.0"
+               iyy="1.0e-06" iyz="0.0"
+               izz="1.0e-06" />
     </inertial>
   </link>
@@ -227,11 +227,11 @@
       <material name="red"/>
      </visual>
-    <inertial>
+<!--    <inertial>
       <origin xyz="0 0 0" />
-      <mass value="1.0e-03" />
-      <inertia ixx="1.0e-03" ixy="0.0" ixz="0.0"
-               iyy="1.0e-03" iyz="0.0"
-               izz="1.0e-03" />
-    </inertial>
+      <mass value="1.0e-04" />
+      <inertia ixx="1.0e-04" ixy="0.0" ixz="0.0"
+               iyy="1.0e-04" iyz="0.0"
+               izz="1.0e-04" />
+    </inertial>-->
   </link>
   </xacro:macro>

Commit message: set moveit pkg
Signed-off-by: Hye-jong KIM <hjkim@robotis.com>

File: turtlebot3_manipulation_description/ros2_control/turtlebot3_manipulation_system.ros2_control.xacro (robot description, xacro)
@@ -91,4 +91,5 @@
         </command_interface>
         <state_interface name="position"/>
+        <state_interface name="velocity"/>
       </joint>
       <joint name="${prefix}gripper_right_joint">
@@ -100,7 +101,5 @@
         </command_interface>
         <state_interface name="position"/>
-      </joint>
-      <joint name="${prefix}end_effector_joint">
-        <state_interface name="position"/>
+        <state_interface name="velocity"/>
       </joint>
     </ros2_control>

Commit message: Added tags
Signed-off-by: Darby Lim <thlim@robotis.com>

File: turtlebot3_manipulation_description/ros2_control/turtlebot3_manipulation_system.ros2_control.xacro (robot description, xacro)
@@ -102,3 +102,6 @@
         <state_interface name="position"/>
         <state_interface name="velocity"/>
+      </joint>
+    </ros2_control>
+  </xacro:macro>
 </robot>

Commit message: Deleted unused args
Signed-off-by: Darby Lim <thlim@robotis.com>

File: turtlebot3_manipulation_description/ros2_control/turtlebot3_manipulation_system.ros2_control.xacro (robot description, xacro)
@@ -6,5 +6,5 @@
 -->
 <robot xmlns:xacro="http://www.ros.org/wiki/xacro">
-  <xacro:macro name="turtlebot3_manipulation_system" params="name prefix use_sim:=^|false use_fake_hardware:=^|false fake_sensor_commands:=^|false slowdown:=2.0">
+  <xacro:macro name="turtlebot3_manipulation_system" params="name prefix use_sim:=^|false use_fake_hardware:=^|false fake_sensor_commands:=^|false">
     <ros2_control name="${name}" type="system">
       <xacro:if value="$(arg use_sim)">

File: turtlebot3_manipulation_description/urdf/turtlebot3_manipulation.urdf.xacro (robot description, xacro)
@@ -6,5 +6,4 @@
   <xacro:arg name="use_fake_hardware" default="false" />
   <xacro:arg name="fake_sensor_commands" default="false" />
-  <xacro:arg name="slowdown" default="2.0" />
   <!-- Import materials macro -->
   <xacro:include filename="$(find turtlebot3_manipulation_description)/gazebo/materials.xacro" />
@@ -32,6 +31,5 @@
     name="TurtleBot3ManipulationSystem" prefix="$(arg prefix)" use_sim="$(arg use_sim)"
     use_fake_hardware="$(arg use_fake_hardware)"
-    fake_sensor_commands="$(arg fake_sensor_commands)"
-    slowdown="$(arg slowdown)"/>
+    fake_sensor_commands="$(arg fake_sensor_commands)"/>
   <gazebo>
     <plugin name="gazebo_ros2_control" filename="libgazebo_ros2_control.so">
