Commit message: setting arm friction

File: turtlebot3_lime_description/gazebo/open_manipulator_sara.gazebo.xacro (robot description, xacro)
@@ -17,4 +17,7 @@
       </actuator>
     </transmission>
+    <gazebo reference="${joint}">
+      <implicitSpringDamper>true</implicitSpringDamper>
+    </gazebo>
   </xacro:macro>
   <xacro:macro name="Link" params="reference">
@@ -34,4 +37,6 @@
   <xacro:Link reference="${prefix}link4"/>
   <xacro:Link reference="${prefix}link5"/>
+  <xacro:Link reference="${prefix}link6"/>
+  <xacro:Link reference="${prefix}link7"/>
   <xacro:Link reference="${prefix}gripper_left_link"/>
   <xacro:Link reference="${prefix}gripper_right_link"/>

File: turtlebot3_lime_description/gazebo/turtlebot3_bigwheel_orin.gazebo.xacro (robot description, xacro)
@@ -13,6 +13,6 @@
     </gazebo>
     <gazebo reference="${prefix}wheel_left_link">
-      <mu1>0.3</mu1>
-      <mu2>0.3</mu2>
+      <mu1>1.0</mu1>
+      <mu2>1.0</mu2>
       <kp>500000.0</kp>
       <kd>10.0</kd>
@@ -23,6 +23,6 @@
     </gazebo>
     <gazebo reference="${prefix}wheel_right_link">
-      <mu1>0.3</mu1>
-      <mu2>0.3</mu2>
+      <mu1>1.0</mu1>
+      <mu2>1.0</mu2>
       <kp>500000.0</kp>
       <kd>10.0</kd>

File: turtlebot3_lime_description/urdf/open_manipulator_sara.urdf.xacro (robot description, xacro)
@@ -34,5 +34,5 @@
       <axis xyz="0 0 1"/>
       <limit velocity="4.8" effort="1" lower="${-pi*0.9}" upper="${pi*0.9}" />
-      <dynamics damping="0.1"/>
+      <dynamics damping="0.7" friction="1.0"/>
     </joint>
     <link name="${prefix}link2">
@@ -62,5 +62,5 @@
       <axis xyz="0 1 0"/>
       <limit velocity="4.8" effort="1" lower="${-pi*0.65}" upper="${pi*0.67}" />
-      <dynamics damping="0.1"/>
+      <dynamics damping="0.7" friction="1.0"/>
     </joint>
     <link name="${prefix}link3">
@@ -90,5 +90,5 @@
       <axis xyz="0 1 0"/>
       <limit velocity="4.8" effort="1" lower="${-pi*0.60}" upper="${pi*0.68}" />
-      <dynamics damping="0.1"/>
+      <dynamics damping="0.7" friction="1.0"/>
     </joint>
     <link name="${prefix}link4">
@@ -118,5 +118,5 @@
       <axis xyz="0 0 1"/>
       <limit velocity="4.8" effort="1" lower="${-pi*0.9}" upper="${pi*0.9}" />
-      <dynamics damping="0.1"/>
+      <dynamics damping="0.7" friction="1.0"/>
     </joint>
     <link name="${prefix}link5">
@@ -146,5 +146,5 @@
       <axis xyz="0 1 0"/>
       <limit velocity="4.8" effort="1" lower="${-pi*0.63}" upper="${pi*0.67}" />
-      <dynamics damping="0.1"/>
+      <dynamics damping="0.7" friction="1.0"/>
     </joint>
     <link name="${prefix}link6">
@@ -179,5 +179,5 @@
       <axis xyz="0 0 1"/>
       <limit velocity="4.8" effort="1" lower="${-pi*0.9}" upper="${pi*0.9}" />
-      <dynamics damping="0.1"/>
+      <dynamics damping="0.7" friction="1.0"/>
     </joint>
     <link name="${prefix}link7">
@@ -187,5 +187,5 @@
           <mesh filename="${meshes_file_direction}/link7.stl" scale="0.001 0.001 0.001"/>
         </geometry>
-        <!-- <material name="grey"/> -->
+        <material name="grey"/>
       </visual>
       <collision>
@@ -227,5 +227,5 @@
       <axis xyz="0 1 0"/>
       <limit velocity="4.8" effort="1" lower="-0.010" upper="0.019" />
-      <dynamics damping="0.1"/>
+      <dynamics damping="0.7" friction="1.0"/>
     </joint>
     <link name="${prefix}gripper_right_link">
@@ -256,5 +256,5 @@
       <limit velocity="4.8" effort="1" lower="-0.010" upper="0.019" />
       <mimic joint="${prefix}gripper_left_joint" multiplier="1"/>
-      <dynamics damping="0.1"/>
+      <dynamics damping="0.7" friction="1.0"/>
     </joint>
     <joint name="${prefix}end_effector_joint" type="fixed">

File: turtlebot3_lime_description/urdf/turtlebot3_bigwheel_orin.urdf.xacro (robot description, xacro)
@@ -40,4 +40,7 @@
       <origin xyz="0.0 0.147125 0.0" rpy="-1.57 0 0"/>
       <axis xyz="0 0 1"/>
+      <!--XM430-W210-->
+      <limit velocity="8.063" effort="3.0"/>
+      <dynamics damping="0.7" friction="1.0"/>
     </joint>
     <link name="${prefix}wheel_left_link">
@@ -66,4 +69,6 @@
       <origin xyz="0.0 -0.147125 0.0" rpy="-1.57 0 0"/>
       <axis xyz="0 0 1"/>
+      <!--XM430-W210-->
+      <limit velocity="8.063" effort="3.0"/>
     </joint>
     <link name="${prefix}wheel_right_link">
@@ -153,7 +158,7 @@
       </visual>
       <collision>
-        <origin xyz="0.0 0 -0.0065" rpy="0 0 0"/>
+        <origin xyz="0.0 0 -0.0111" rpy="0 0 0"/>
         <geometry>
-          <cylinder length="0.0315" radius="0.055"/>
+          <cylinder length="0.0378" radius="0.025"/>
         </geometry>
       </collision>
