Commit message: modify joint limit

File: turtlebot3_lime_description/urdf/open_manipulator_sara.urdf.xacro (robot description, xacro)
@@ -61,5 +61,5 @@
       <origin xyz="0.0 0.0 0.0595" rpy="0 0 0"/>
       <axis xyz="0 1 0"/>
-      <limit velocity="4.8" effort="1" lower="${-pi*0.65}" upper="${pi*0.67}" />
+      <limit velocity="4.8" effort="1" lower="${-pi*0.541}" upper="${pi*0.562}" />
       <dynamics damping="0.7" friction="1.0"/>
     </joint>
@@ -89,5 +89,5 @@
       <origin xyz="0.0 0 0.124" rpy="0 0 0"/>
       <axis xyz="0 1 0"/>
-      <limit velocity="4.8" effort="1" lower="${-pi*0.60}" upper="${pi*0.68}" />
+      <limit velocity="4.8" effort="1" lower="${-pi*0.560}" upper="${pi*0.591}" />
       <dynamics damping="0.7" friction="1.0"/>
     </joint>
@@ -117,5 +117,5 @@
       <origin xyz="0.0 0.0 0.045" rpy="0 0 0"/>
       <axis xyz="0 0 1"/>
-      <limit velocity="4.8" effort="1" lower="${-pi*0.9}" upper="${pi*0.9}" />
+      <limit velocity="4.8" effort="1" lower="${-pi*0.5}" upper="${pi*0.5}" />
       <dynamics damping="0.7" friction="1.0"/>
     </joint>
@@ -145,5 +145,5 @@
       <origin xyz="0.0 0.0 0.0595" rpy="0 0 0"/>
       <axis xyz="0 1 0"/>
-      <limit velocity="4.8" effort="1" lower="${-pi*0.63}" upper="${pi*0.67}" />
+      <limit velocity="4.8" effort="1" lower="${-pi*0.531}" upper="${pi*0.567}" />
       <dynamics damping="0.7" friction="1.0"/>
     </joint>

Commit message: modify parameters

File: turtlebot3_lime_description/urdf/open_manipulator_sara.urdf.xacro (robot description, xacro)
@@ -229,24 +229,11 @@
       <dynamics damping="0.7" friction="1.0"/>
     </joint>
-    <link name="${prefix}gripper_right_link">
-      <visual>
-        <origin xyz="0 0 0" rpy="0 0 0"/>
-        <geometry>
-          <mesh filename="${meshes_file_direction}/gripper_right_palm.stl" scale="0.001 0.001 0.001"/>
-        </geometry>
-        <material name="grey"/>
-      </visual>
-      <collision>
-        <origin xyz="0 0 0" rpy="0 0 0"/>
-        <geometry>
-          <mesh filename="${meshes_file_direction}/gripper_right_palm.stl" scale="0.001 0.001 0.001"/>
-        </geometry>
-      </collision>
-      <inertial>
-        <origin xyz="0 0 0" />
-        <mass value="1.0e-03" />
-        <inertia ixx="1.0e-03" ixy="0.0" ixz="0.0" iyy="1.0e-03" iyz="0.0" izz="1.0e-03" />
-      </inertial>
-    </link>
+    <!-- Move it 2 not find mimic-->
+    <!-- https://github.com/ROBOTIS-GIT/turtlebot3_lime/issues/66  -->
+    <joint name="${prefix}gripper_right_joint_mimic" type="fixed">
+      <parent link="${prefix}link7" />
+      <child link="dummy_mimic_fix" />
+    </joint>
+    <link name="dummy_mimic_fix"/>
     <joint name="${prefix}gripper_right_joint" type="prismatic">
       <parent link="${prefix}link7"/>
@@ -258,4 +245,24 @@
       <dynamics damping="0.7" friction="1.0"/>
     </joint>
+    <link name="${prefix}gripper_right_link">
+      <visual>
+        <origin xyz="0 0 0" rpy="0 0 0"/>
+        <geometry>
+          <mesh filename="${meshes_file_direction}/gripper_right_palm.stl" scale="0.001 0.001 0.001"/>
+        </geometry>
+        <material name="grey"/>
+      </visual>
+      <collision>
+        <origin xyz="0 0 0" rpy="0 0 0"/>
+        <geometry>
+          <mesh filename="${meshes_file_direction}/gripper_right_palm.stl" scale="0.001 0.001 0.001"/>
+        </geometry>
+      </collision>
+      <inertial>
+        <origin xyz="0 0 0" />
+        <mass value="1.0e-03" />
+        <inertia ixx="1.0e-03" ixy="0.0" ixz="0.0" iyy="1.0e-03" iyz="0.0" izz="1.0e-03" />
+      </inertial>
+    </link>
     <joint name="${prefix}end_effector_joint" type="fixed">
       <origin xyz="0.0 0.0 0.115" rpy="0 0 0"/>
@@ -277,11 +284,4 @@
       </inertial>
     </link>
-    <!-- Move it 2 not find mimic-->
-    <!-- https://github.com/ROBOTIS-GIT/turtlebot3_lime/issues/66  -->
-    <joint name="${prefix}gripper_right_joint_mimic" type="fixed">
-      <parent link="${prefix}link7" />
-      <child link="dummy_mimic_fix" />
-    </joint>
-    <link name="dummy_mimic_fix"/>
   </xacro:macro>
 </robot>
